File: KiCAD/Air Monitor.kicad_sch (KiCad schematic)
At the start: 16 parts, among them J1 Barrel_Jack, U1 ESP32-DevKitC, U2 BME680, U3 SGP40

Commit message: PCB updates
Parts:
- added C7: 10μF, Capacitor_SMD:C_0402_1005Metric, symbol Device:C
- added C8: 1μF, Capacitor_SMD:C_0402_1005Metric, symbol Device:C
- added J2: USB_B_Micro, Connector_USB:USB_Micro-B_Wuerth_629105150521, symbol Connector:USB_B_Micro
- added JP1: SolderJumper_2_Open, Jumper:SolderJumper-2_P1.3mm_Open_RoundedPad1.0x1.5mm, symbol Jumper:SolderJumper_2_Open
- added U4: LM66100DCK, Package_TO_SOT_SMD:SOT-363_SC-70-6, symbol Power_Management:LM66100DCK
- J1: footprint Connector_BarrelJack:BarrelJack_SwitchcraftConxall_RAPC10U_Horizontal -> Connector_BarrelJack:BarrelJack_Wuerth_6941xx301002; symbol Connector:Barrel_Jack -> Connector:Barrel_Jack_Switch
Connections:
- net +5V: now also C7.2, JP1.2 (B), U4.3 (~{CE}), U4.6 (VOUT); no longer C2.2, J1.1
- net GND: now also J1.3, C7.1, C8.1, J2.5 (GND), J2.SH (Shield), U4.2 (GND), U4.5 (ST)
- net ESP 5V Pin: now reaches U1.19 (5V)
- net ESP 5V Pin: now also C2.2, JP1.1 (A)
- net SGP VDD: now reaches C6.1, R5.1, U3.1 (VDD)
- new net 5V INPUT: C8.2, J1.1, J2.1 (VBUS), U4.1 (VIN)
Other:
- note added: "5V POWER SUPPLY"
- note added: "ESP32"
- note added: "SPS30 CONNECTOR"
- note removed: "SPS30 CONNECTOR & POWER SUPPLY"
- moved on the sheet: C1, R4, SPS30
